File: PCB/rp2040 led.kicad_sch (KiCad schematic)
At the start: 38 parts, among them J1 Conn_01x03_Pin, J2 Conn_01x20_Pin, J3 Conn_01x20_Pin, J4 USB_C_Receptacle_USB2.0_16P, SW1 SW_Push, U1 RP2040, U2 MCP1700x-120xxTT, U3 W25Q128JVS, Y1 12MHz

Commit message: converting to newer version
Other:
- moved on the sheet: C10, C11, C12

Commit message: WS2812B
Parts:
- removed D1, D2, D3, D4: SK6812MINI, LED_SMD:LED_SK6812MINI_PLCC4_3.5x3.5mm_P1.75mm, symbol LED:SK6812MINI
- added D1, D2, D3, D4: WS2812B, LED_SMD:LED_WS2812B_PLCC4_5.0x5.0mm_P3.2mm, symbol LED:WS2812B
Connections:
- net +3V3: now also D1.3 (VSS), D2.3 (VSS), D3.3 (VSS), D4.3 (VSS)
- net GND: now also D1.1 (VDD), D2.1 (VDD), D3.1 (VDD), D4.1 (VDD)
- net GPIO22: now also D1.4 (DIN)
- new net: D3.2 (DOUT), D4.4 (DIN)
- new net: D2.2 (DOUT), D3.4 (DIN)
- new net: D1.2 (DOUT), D2.4 (DIN)
