File: PCB/rp2040 led.kicad_pcb (KiCad board)
At the start: 2 copper layers, 31 x 51.5 mm, 40 parts, among them J1 Conn_01x03_Pin, J2 Conn_01x20_Pin, J3 Conn_01x20_Pin, J4 USB_C_Receptacle_USB2.0_16P, SW1 SW_Push, U1 RP2040, U2 MCP1700x-120xxTT, U3 W25Q128JVS, Y1 12MHz

Commit message: WS2812B
Parts:
- D1, D2, D3, D4: value SK6812MINI -> WS2812B; footprint LED_SMD:LED_SK6812MINI_PLCC4_3.5x3.5mm_P1.75mm -> LED_SMD:LED_WS2812B_PLCC4_5.0x5.0mm_P3.2mm
- moved D4 7.98 mm to (97.5, 76.0)
- moved D3 5.60 mm to (105.0, 76.0)
- moved D1 2.96 mm to (97.5, 70.0)
- moved D2 2.28 mm to (105.0, 70.0)
- moved J1 0.85 mm to (105.3, 65.4)
Connections:
- D1 pad 1: Net-(D1-DOUT) -> GND
- D1 pad 2: +3V3 -> Net-(D1-DOUT)
- D1 pad 3: GPIO22 -> +3V3
- D1 pad 4: GND -> GPIO22
- D2 pad 1: Net-(D2-DOUT) -> GND
- D2 pad 2: +3V3 -> Net-(D2-DOUT)
- D2 pad 3: Net-(D1-DOUT) -> +3V3
- D2 pad 4: GND -> Net-(D1-DOUT)
- D3 pad 1: Net-(D3-DOUT) -> GND
- D3 pad 2: +3V3 -> Net-(D3-DOUT)
- D3 pad 3: Net-(D2-DOUT) -> +3V3
- D3 pad 4: GND -> Net-(D2-DOUT)
- D4 pad 1: unconnected-(D4-DOUT-Pad1) -> GND
- D4 pad 2: +3V3 -> unconnected-(D4-DOUT-Pad2)
- D4 pad 3: Net-(D3-DOUT) -> +3V3
- D4 pad 4: GND -> Net-(D3-DOUT)
Routing:
- net +3V3: track 153.5 -> 171.9 mm, vias 11 -> 14
- net Net-(D3-DOUT): track 10.2 -> 4.38 mm
- net Net-(D2-DOUT): track 11.6 -> 6.30 mm, vias 2 -> 0
- net Net-(D1-DOUT): track 10.2 -> 14.6 mm
- net GPIO22: track 29.3 -> 27.8 mm
- net SWD: track 16.9 -> 15.9 mm
- net GND: vias 65 -> 74

Commit message: stitching groung planes
Parts:
- moved G*** 0.50 mm to (90.5, 73.4)
Routing:
- net GND: vias 74 -> 122
