File: PCB/rp2040 led.kicad_pcb (KiCad board)
At the start: 2 copper layers, 31 x 51.5 mm, 40 parts, among them J1 Conn_01x03_Pin, J2 Conn_01x20_Pin, J3 Conn_01x20_Pin, J4 USB_C_Receptacle_USB2.0_16P, SW1 SW_Push, U1 RP2040, U2 MCP1700x-120xxTT, U3 W25Q128JVS, Y1 12MHz

Commit message: updated the images.
Routing:
- net GND: vias 122 -> 129
Changed lines of the file:
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@@
+	)
+	(via
+		(at 105.2 51.8)
+		(size 0.6)
+		(drill 0.3)
+		(layers "F.Cu" "B.Cu")
+		(free yes)
+		(net "GND")
+	)
+	(via
+		(at 104.1 77.9)
+		(size 0.6)
+		(drill 0.3)
+		(layers "F.Cu" "B.Cu")
+		(free yes)
+		(net "GND")
 	)
 	(via
@@
 	)
 	(via
+		(at 105.8 34.3)
+		(size 0.6)
+		(drill 0.3)
+		(layers "F.Cu" "B.Cu")
+		(free yes)
+		(net "GND")
+	)
+	(via
 		(at 97.3 31)
 		(size 0.6)
@@
 	)
 	(via
+		(at 88.1 68.7)
+		(size 0.6)
+		(drill 0.3)
+		(layers "F.Cu" "B.Cu")
+		(free yes)
+		(net "GND")
+	)
+	(via
 		(at 91.4 48.4)
 		(size 0.6)
@@
 	)
 	(via
+		(at 105.1 40.6)
+		(size 0.6)
+		(drill 0.3)
+		(layers "F.Cu" "B.Cu")
+		(free yes)
+		(net "GND")
+	)
+	(via
 		(at 86.4 73.6)
 		(size 0.6)
@@
 	)
 	(via
+		(at 109 41.1)
+		(size 0.6)
+		(drill 0.3)
+		(layers "F.Cu" "B.Cu")
+		(free yes)
+		(net "GND")
+	)
+	(via
 		(at 86.1 78.4)
 		(size 0.6)
@@
 		(net "GND")
 	)
+	(via
+		(at 86.2 70)
+		(size 0.6)
+		(drill 0.3)
+		(layers "F.Cu" "B.Cu")
+		(free yes)
+		(net "GND")
+	)
